File: 1.kicad_pcb (KiCad board)
At the start: 2 copper layers, 154 x 123 mm, 61 parts, among them Q1 BC547, SW1 SW_SPDT, SW2 SW_DPST_x2, U1 NE555P, U2 74HC595, U3 ULN2803A, U5 TSR_1-2450

Commit message: izmena
Parts:
- removed REF** (x4): MountingHole_3.2mm_M3, MountingHole:MountingHole_3.2mm_M3
- BT1: renamed from + BT1 -; value + Battery_Cell - -> Battery_Cell
