File: 1.kicad_sch (KiCad schematic)
At the start: 57 parts, among them Q1 BC547, SW1 SW_SPDT, SW2 SW_DPST_x2, U1 NE555P, U2 74HC595, U3 ULN2803A, U5 TSR_1-2450

Commit message: izmena
Changed lines of the file:
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@@
+		)
+	)
+	(label "Izmena"
+		(at 139.7 44.45 0)
+		(effects
+			(font
+				(size 3.81 3.81)
+			)
+			(justify left bottom)
 		)
 	)
